File: BatteryPod.kicad_sch (KiCad schematic)
At the start: 25 parts, among them J1 VIN, U1 LM5157RTER

Commit message: feat: fully routed USB-PD, new lower profile inductor
Parts:
- added JP1: EN_SEL, Connector_PinHeader_2.54mm:PinHeader_1x03_P2.54mm_Vertical, symbol Jumper:Jumper_3_Open
- L1: value SER2918H-333KL -> CDEP15D90T150NP-220MC; footprint IND_SER2918H_COC -> Sumida:CDEP15D90T150NP-220MC; Part C3911813 -> C171581
- R4: value 63.4K -> 1.21K; Part C218107 -> C705737
- TP1, TP2: now not fitted
Connections:
- net +BATT: now also JP1.3 (B)
- net REG_EN: now also JP1.2 (C); no longer R5.1
- new net PD_READY: JP1.1 (A), R5.1
Changed lines of the file:
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@@
 	(wire
 		(pts
+			(xy 127 123.19) (xy 127 121.92)
+		)
+		(stroke
+			(width 0)
+			(type default)
+		)
+	)
+	(wire
+		(pts
 			(xy 161.29 93.98) (xy 166.37 93.98)
 		)
@@
 	(wire
 		(pts
+			(xy 128.27 123.19) (xy 127 123.19)
+		)
+		(stroke
+			(width 0)
+			(type default)
+		)
+	)
+	(wire
+		(pts
 			(xy 96.52 116.84) (xy 96.52 114.3)
 		)
@@
 		)
 	)
+	(label "PD_READY"
+		(at 113.03 138.43 0)
+		(fields_autoplaced yes)
+		(effects
+			(font
+				(size 1.27 1.27)
+			)
+			(justify left bottom)
+		)
+	)
 	(label "FB"
 		(at 161.29 96.52 0)
@@
 		)
 	)
-	(label "SW"
-		(at 222.25 80.01 180)
+	(label "PD_READY"
+		(at 120.65 118.11 180)
 		(fields_autoplaced yes)
 		(effects
@@
 		)
 	)
-	(label "REG_EN"
-		(at 113.03 138.43 0)
+	(label "SW"
+		(at 222.25 80.01 180)
 		(fields_autoplaced yes)
 		(effects
@@
 				(size 1.27 1.27)
 			)
-			(justify left bottom)
+			(justify right bottom)
 		)
 	)
@@
 		)
 	)
+	(label "REG_EN"
+		(at 128.27 123.19 0)
+		(fields_autoplaced yes)
+		(effects
+			(font
+				(size 1.27 1.27)
+			)
+			(justify left bottom)
+		)
+	)
 	(symbol
 		(lib_id "power:GND")
@@
 	)
 	(symbol
+		(lib_id "Jumper:Jumper_3_Open")
+		(at 127 118.11 0)
+		(unit 1)
+		(exclude_from_sim yes)
+		(in_bom no)
+		(on_board yes)
+		(dnp no)
+		(fields_autoplaced yes)
+		(property "Reference" "JP1"
+			(at 127 111.76 0)
+			(effects
+				(font
+					(size 1.27 1.27)
+				)
+			)
+		)
+		(property "Value" "EN_SEL"
+			(at 127 114.3 0)
+			(effects
+				(font
+					(size 1.27 1.27)
+				)
+			)
+		)
+		(property "Footprint" "Connector_PinHeader_2.54mm:PinHeader_1x03_P2.54mm_Vertical"
+			(at 127 118.11 0)
+			(effects
+				(font
+					(size 1.27 1.27)
+				)
+				(hide yes)
+			)
+		)
+		(property "Datasheet" "~"
+			(at 127 118.11 0)
+			(effects
+				(font
+					(size 1.27 1.27)
+				)
+				(hide yes)
+			)
+		)
+		(property "Description" "Jumper, 3-pole, both open"
+			(at 127 118.11 0)
+			(effects
+				(font
+					(size 1.27 1.27)
+				)
+				(hide yes)
+			)
+		)
+		(pin "2"
+		)
+		(pin "3"
+		)
+		(pin "1"
+		)
+		(instances
+			(project "BatteryPod"
+				(path "/4321c496-0c88-4f4f-a1d3-dd2bca7d98aa"
+					(reference "JP1")
+					(unit 1)
+				)
+			)
+		)
+	)
+	(symbol
 		(lib_id "power:GND")
 		(at 90.17 91.44 270)
@@
 	)
 	(symbol
+		(lib_id "power:+BATT")
+		(at 133.35 118.11 270)
+		(unit 1)
+		(exclude_from_sim no)
+		(in_bom yes)
+		(on_board yes)
+		(dnp no)
+		(fields_autoplaced yes)
+		(property "Reference" "#PWR028"
+			(at 129.54 118.11 0)
+			(effects
+				(font
+					(size 1.27 1.27)
+				)
+				(hide yes)
+			)
+		)
+		(property "Value" "+BATT"
+			(at 137.16 118.1099 90)
+			(effects
+				(font
+					(size 1.27 1.27)
+				)
+				(justify left)
+			)
+		)
+		(property "Footprint" ""
+			(at 133.35 118.11 0)
+			(effects
+				(font
+					(size 1.27 1.27)
+				)
+				(hide yes)
+			)
+		)
+		(property "Datasheet" ""
+			(at 133.35 118.11 0)
+			(effects
+				(font
+					(size 1.27 1.27)
+				)
+				(hide yes)
+			)
+		)
+		(property "Description" "Power symbol creates a global label with name \"+BATT\""
+			(at 133.35 118.11 0)
+			(effects
+				(font
+					(size 1.27 1.27)
+				)
+				(hide yes)
+			)
+		)
+		(pin "1"
+		)
+		(instances
+			(project "BatteryPod"
+				(path "/4321c496-0c88-4f4f-a1d3-dd2bca7d98aa"
+					(reference "#PWR028")
+					(unit 1)
+				)
+			)
+		)
+	)
+	(symbol
 		(lib_id "power:GND")
 		(at 90.17 86.36 270)
@@
 		(in_bom no)
 		(on_board yes)
-		(dnp no)
+		(dnp yes)
 		(fields_autoplaced yes)
 		(property "Reference" "TP1"
@@
 			)
 		)
-		(property "Value" "SER2918H-333KL"
+		(property "Value" "CDEP15D90T150NP-220MC"
 			(at 209.55 82.55 0)
 			(effects
@@
 			)
 		)
-		(property "Footprint" "IND_SER2918H_COC"
+		(property "Footprint" "Sumida:CDEP15D90T150NP-220MC"
 			(at 201.93 80.01 0)
 			(effects
@@
 			)
 		)
-		(property "Part" "C3911813"
-			(at 201.93 80.01 0)
-			(effects
-				(font
-					(size 1.27 1.27)
-				)
-				(hide yes)
-			)
-		)
-		(property "Part#" ""
+		(property "Part" "C171581"
 			(at 201.93 80.01 0)
 			(effects
@@
 		(in_bom no)
 		(on_board yes)
-		(dnp no)
+		(dnp yes)
 		(fields_autoplaced yes)
 		(property "Reference" "TP2"
@@
 			)
 		)
-		(property "Value" "63.4K"
+		(property "Value" "1.21K"
 			(at 105.156 108.966 0)
 			(effects
@@
 			)
 		)
-		(property "Part" "C218107"
-			(at 102.87 107.95 0)
-			(effects
-				(font
-					(size 1.27 1.27)
-				)
-				(hide yes)
-			)
-		)
-		(property "Part#" ""
+		(property "Part" "C705737"
 			(at 102.87 107.95 0)
 			(effects

Commit message: patch: final trace cleaups/parameter updates
Parts:
- C3: value 0.1uF -> 1uF; Part C597287 -> C342988
Connections:
- net GND: now also U1.15 (NC)
Changed lines of the file:
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@@
+	)
+	(junction
+		(at 163.83 78.74)
+		(diameter 0)
+		(color 0 0 0 0)
 	)
 	(junction
@@
 	)
 	(junction
-		(at 163.83 77.47)
-		(diameter 0)
-		(color 0 0 0 0)
-	)
-	(junction
 		(at 95.25 76.2)
 		(diameter 0)
@@
 	(wire
 		(pts
-			(xy 163.83 76.2) (xy 163.83 77.47)
-		)
-		(stroke
-			(width 0)
-			(type default)
-		)
-	)
-	(wire
-		(pts
 			(xy 102.87 114.3) (xy 96.52 114.3)
 		)
@@
 	(wire
 		(pts
+			(xy 161.29 81.28) (xy 163.83 81.28)
+		)
+		(stroke
+			(width 0)
+			(type default)
+		)
+	)
+	(wire
+		(pts
 			(xy 90.17 81.28) (xy 105.41 81.28)
 		)
@@
 	(wire
 		(pts
-			(xy 166.37 77.47) (xy 163.83 77.47)
+			(xy 166.37 78.74) (xy 163.83 78.74)
 		)
 		(stroke
@@
 	(wire
 		(pts
-			(xy 163.83 78.74) (xy 163.83 77.47)
+			(xy 163.83 76.2) (xy 163.83 78.74)
 		)
 		(stroke
@@
 		(pts
 			(xy 46.99 116.84) (xy 46.99 114.3)
+		)
+		(stroke
+			(width 0)
+			(type default)
+		)
+	)
+	(wire
+		(pts
+			(xy 163.83 81.28) (xy 163.83 78.74)
 		)
 		(stroke
@@
 			)
 		)
-		(property "Part#" ""
-			(at 210.82 119.38 0)
-			(effects
-				(font
-					(size 1.27 1.27)
-				)
-				(hide yes)
-			)
-		)
 		(pin "2"
 		)
@@
 			)
 		)
-		(property "Value" "0.1uF"
+		(property "Value" "1uF"
 			(at 106.934 77.724 90)
 			(effects
@@
 			)
 		)
-		(property "Part" "C597287"
+		(property "Part" "C342988"
 			(at 100.33 78.74 90)
 			(effects
@@
 	(symbol
 		(lib_id "power:GND")
-		(at 166.37 77.47 90)
+		(at 166.37 78.74 90)
 		(unit 1)
 		(exclude_from_sim no)
@@
 		(fields_autoplaced yes)
 		(property "Reference" "#PWR01"
-			(at 172.72 77.47 0)
+			(at 172.72 78.74 0)
 			(effects
 				(font
@@
 		)
 		(property "Value" "GND"
-			(at 170.18 77.4699 90)
+			(at 170.18 78.7399 90)
 			(effects
 				(font
@@
 		)
 		(property "Footprint" ""
-			(at 166.37 77.47 0)
+			(at 166.37 78.74 0)
 			(effects
 				(font
@@
 		)
 		(property "Datasheet" ""
-			(at 166.37 77.47 0)
+			(at 166.37 78.74 0)
 			(effects
 				(font
@@
 		)
 		(property "Description" "Power symbol creates a global label with name \"GND\" , ground"
-			(at 166.37 77.47 0)
-			(effects
-				(font
+			(at 166.37 78.74 0)
+			(effects
+				(font
